Commit message: Task A.3 complete. Created yaml file and added parameters to urdf

File: nuturtle_description/urdf/turtlebot3_burger.urdf.xacro (robot description, xacro)
@@ -1,7 +1,18 @@
 <?xml version="1.0" ?>
 <!-- Modified the package to nuturtle_description -->
+<!-- Added the properties from the yaml file -->
 <robot name="turtlebot3_burger" xmlns:xacro="http://ros.org/wiki/xacro">
   <!-- <xacro:include filename="$(find nuturtle_description)/urdf/common_properties.xacro"/> -->
   <!-- <xacro:include filename="$(find nuturtle_description)/urdf/turtlebot3_burger.gazebo.xacro"/> -->
+  <xacro:property name="yaml_file" value="$(find nuturtle_description)/config/diff_params.yaml" />
+  <xacro:property name="props" value="${xacro.load_yaml(yaml_file)}" />
+  <xacro:property name="ros_params" value="${props['/**']}"/>
+  <xacro:property name="params" value="${ros_params['ros__parameters']}"/>
+  <xacro:property name="wheel_radius"  value="${params['wheel_radius']}" />
+  <xacro:property name="track_width"  value="${params['track_width']}" />
+  <xacro:property name="motor_cmd_max"  value="${params['motor_cmd_max']}" />
+  <xacro:property name="motor_cmd_per_rad_sec"  value="${params['motor_cmd_per_rad_sec']}" />
+  <xacro:property name="encoder_ticks_per_rad"  value="${params['encoder_ticks_per_rad']}" />
+  <xacro:property name="collision_radius"  value="${params['collision_radius']}" />
   <link name="base_footprint"/>
   <joint name="base_joint" type="fixed">
@@ -21,5 +32,12 @@
       <origin xyz="-0.032 0 0.070" rpy="0 0 0"/>
       <geometry>
-        <box size="0.140 0.140 0.143"/>
+        <!-- If collision_radius is Lower Than 0.0, use the original box collision geometry -->
+        <xacro:if value = "${collision_radius &lt; 0.0}">
+          <box size="0.140 0.140 0.143"/>
+        </xacro:if>
+        <!-- Otherwise, the cylinder should be the same height as the box it is replacing -->
+        <xacro:if value = "${collision_radius &gt; 0.0}">
+          <cylinder length="0.143" radius="${collision_radius}"/>
+        </xacro:if>
       </geometry>
     </collision>
@@ -35,5 +53,5 @@
     <parent link="base_link"/>
     <child link="wheel_left_link"/>
-    <origin xyz="0.0 0.08 0.023" rpy="-1.57 0 0"/>
+    <origin xyz="0.0 ${track_width/2} 0.023" rpy="-1.57 0 0"/>
     <axis xyz="0 0 1"/>
   </joint>
@@ -49,5 +67,5 @@
       <origin xyz="0 0 0" rpy="0 0 0"/>
       <geometry>
-        <cylinder length="0.018" radius="0.033"/>
+        <cylinder length="0.018" radius="${wheel_radius}"/>
       </geometry>
     </collision>
@@ -63,5 +81,5 @@
     <parent link="base_link"/>
     <child link="wheel_right_link"/>
-    <origin xyz="0.0 -0.080 0.023" rpy="-1.57 0 0"/>
+    <origin xyz="0.0 -${track_width/2} 0.023" rpy="-1.57 0 0"/>
     <axis xyz="0 0 1"/>
   </joint>
@@ -77,5 +95,5 @@
       <origin xyz="0 0 0" rpy="0 0 0"/>
       <geometry>
-        <cylinder length="0.018" radius="0.033"/>
+        <cylinder length="0.018" radius="${wheel_radius}"/>
       </geometry>
     </collision>

Commit message: URDF defaults the color of base link to purple

File: nuturtle_description/urdf/turtlebot3_burger.urdf.xacro (robot description, xacro)
@@ -1,5 +1,5 @@
 <?xml version="1.0" ?>
 <!-- Modified the package to nuturtle_description -->
-<!-- Added the properties from the yaml file -->
+<!-- Modified to add the properties from the yaml file -->
 <robot name="turtlebot3_burger" xmlns:xacro="http://ros.org/wiki/xacro">
   <!-- <xacro:include filename="$(find nuturtle_description)/urdf/common_properties.xacro"/> -->
@@ -15,4 +15,19 @@
   <xacro:property name="encoder_ticks_per_rad"  value="${params['encoder_ticks_per_rad']}" />
   <xacro:property name="collision_radius"  value="${params['collision_radius']}" />
+  <!-- Colors -->
+  <!-- Northwestern Purple -->
+  <material name="purple">
+    <color rgba="0.3 0.16 0.52 1.0"/>
+  </material>
+  <material name="red">
+    <color rgba="0.9 0 0 1.0"/>
+  </material>
+  <material name="green">
+    <color rgba="0 0.9 0 1.0"/>
+  </material>
+  <material name="blue">
+    <color rgba="0 0 0.9 1.0"/>
+  </material>
+  <xacro:arg name="color" default="purple"/>
   <link name="base_footprint"/>
   <joint name="base_joint" type="fixed">
@@ -27,5 +42,5 @@
         <mesh filename="package://nuturtle_description/meshes/burger_base.stl" scale="0.001 0.001 0.001"/>
       </geometry>
-      <material name="light_black"/>
+      <material name="$(arg color)"/>
     </visual>
     <collision>

Commit message: Task A.5 complete

File: nuturtle_description/urdf/turtlebot3_burger.urdf.xacro (robot description, xacro)
@@ -2,4 +2,5 @@
 <!-- Modified the package to nuturtle_description -->
 <!-- Modified to add the properties from the yaml file -->
+<!-- Modified to add new color options -->
 <robot name="turtlebot3_burger" xmlns:xacro="http://ros.org/wiki/xacro">
   <!-- <xacro:include filename="$(find nuturtle_description)/urdf/common_properties.xacro"/> -->
@@ -29,4 +30,7 @@
   <material name="blue">
     <color rgba="0 0 0.9 1.0"/>
+  </material>
+  <material name="dark">
+    <color rgba="0.25 0.25 0.25 1.0"/>
   </material>
   <link name="base_footprint"/>
